File: BuckLinReg_5V.sch (KiCad schematic (older format))
At the start: 66 parts, among them J1 Barrel_Jack, J2 796638-4, J3 1x2 Male, J4 796634-4, Q1 PMBT2222, Q2 Si4435FDY, SW1 SW_SPDT, U1 TLV76050DBZT, U101 INA180A3IDBVR, U102 TLV7011KCKT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

Commit message: Changed nettie and gnd clearances
Parts:
- D4: footprint Diode_SMD:D_SOD-323_HandSoldering -> Package_TO_SOT_SMD:SOT-23_Handsoldering; MFPN PDZ2.4B,115 -> BZX84-C2V4,215
Changed lines of the file:
@@
 F 0 "D4" V 8454 10105 50  0000 L CNN
 F 1 "2V4" V 8545 10105 50  0000 L CNN
-F 2 "Diode_SMD:D_SOD-323_HandSoldering" H 8500 10025 50  0001 C CNN
-F 3 "https://rocelec.widen.net/view/pdf/girsb18scs/PHGLS19616-1.pdf?t.download=true&u=5oefqw" H 8500 10025 50  0001 C CNN
-F 4 "PDZ2.4B,115" V 8500 10025 50  0001 C CNN "MFPN"
+F 2 "Package_TO_SOT_SMD:SOT-23_Handsoldering" H 8500 10025 50  0001 C CNN
+F 3 "https://rocelec.widen.net/view/pdf/fysgtbvgew/PHGLS29437-1.pdf?t.download=true&u=5oefqw" H 8500 10025 50  0001 C CNN
+F 4 "BZX84-C2V4,215" V 8500 10025 50  0001 C CNN "MFPN"
 	1    8500 10025
 	0    1    1    0

Commit message: PCB v1.1 ordered
Parts:
- Q2: MFPN (none) -> Si4435FDY
- U101: MFPN (none) -> INA180A3IDBVR
- U102: MFPN (none) -> TLV7011DBVR
Changed lines of the file:
@@
 F 2 "Package_SO:SO-8_3.9x4.9mm_P1.27mm" H 5875 2450 50  0001 C CNN
 F 3 "" H 5875 2450 50  0001 C CNN
+F 4 "Si4435FDY" H 5875 2000 50  0001 C CNN "MFPN"
 	1    5875 2000
 	0    -1   -1   0
@@
 F 2 "Package_TO_SOT_SMD:SOT-23-5_HandSoldering" H 6250 9315 60  0001 C CNN
 F 3 "https://www.ti.com/lit/gpn/ina180" H 6250 9856 60  0000 C CNN
+F 4 "INA180A3IDBVR" H 6250 9375 50  0001 C CNN "MFPN"
 	1    6250 9375
 	1    0    0    -1
@@
 F 2 "Package_TO_SOT_SMD:SOT-23-5_HandSoldering" H 8875 9475 50  0001 L CNN
 F 3 "http://www.ti.com/lit/gpn/tlv7011" H 9825 9350 50  0000 C CNN
+F 4 "TLV7011DBVR" H 8975 9675 50  0001 C CNN "MFPN"
 	1    8975 9675
 	1    0    0    -1

Commit message: Prettifying schematic
Parts:
- added TP13, TP15: TestPoint, symbol Connector:TestPoint
Connections:
- net OCP_TRIGGER: now also TP15.1
- net Vo: now also TP13.1
Changed lines of the file:
@@
 Wire Wire Line
 	8500 10225 8500 10275
-Text Label 9275 9675 0    50   ~ 0
+Text Label 9600 9675 0    50   ~ 0
 OCP_TRIGGER
 Wire Wire Line
@@
 	1    0    0    -1
 $EndComp
-Text Notes 6425 10500 0    50   ~ 0
+Text Notes 6650 10550 0    50   ~ 0
 RC time constant of 1 ms to prevent spikes\nshorter than 1-2 ms from tripping OCP
+$Comp
+L Connector:TestPoint TP13
+U 1 1 60871EC0
+P 7425 9175
+F 0 "TP13" H 7483 9293 50  0000 L CNN
+F 1 "TestPoint" H 7483 9202 50  0000 L CNN
+F 2 "" H 7625 9175 50  0001 C CNN
+F 3 "~" H 7625 9175 50  0001 C CNN
+	1    7425 9175
+	1    0    0    -1
+$EndComp
+Connection ~ 7425 9175
+Wire Wire Line
+	9275 9675 9400 9675
+$Comp
+L Connector:TestPoint TP15
+U 1 1 60B92EE2
+P 9400 9550
+F 0 "TP15" H 9458 9668 50  0000 L CNN
+F 1 "TestPoint" H 9458 9577 50  0000 L CNN
+F 2 "" H 9600 9550 50  0001 C CNN
+F 3 "~" H 9600 9550 50  0001 C CNN
+	1    9400 9550
+	1    0    0    -1
+$EndComp
+Wire Wire Line
+	9400 9550 9400 9675
+Connection ~ 9400 9675
+Wire Wire Line
+	9400 9675 9600 9675
 $EndSCHEMATC
